Commit message: urdf: added stylus offset to match actual length and use tip as pointer

File: models/urdf/omni.urdf (robot description, URDF)
Before this commit: robot phantom_omni, 7 links, 6 joints
Joints:
- joint roll: origin xyz=0 -0.023 0 rpy=3.14159 3.14159 0 -> xyz=0 -0.029 0 rpy=3.14159 3.14159 0

Commit message: Removing strange offsets on gimbal joints added to compensate for issues with old Omni I was using.  Tested with newer Ethernet based Touch and everything is now consistent, including URDF

File: models/urdf/omni.urdf (robot description, URDF)
Before this commit: robot phantom_omni, 7 links, 6 joints
Joints:
- joint pitch: origin xyz=0 0.0525 0 rpy=0.5 0 0 -> xyz=0 0.0525 0 rpy=1.5708 0 0
- joint yaw: axis 0 1 0 -> 0 -1 0

Commit message: Release 1.0

File: models/urdf/omni.urdf (robot description, URDF)
Before this commit: robot phantom_omni, 7 links, 6 joints
Links:
- link base: geometry visual mesh filename=package://saw_sensable_phantom_models/meshes/base.stl
- link lower_arm: geometry visual mesh filename=package://saw_sensable_phantom_models/meshes/lower_arm.stl
- link stylus: geometry visual mesh filename=package://saw_sensable_phantom_models/meshes/pen.stl
- link tip: geometry visual mesh filename=package://saw_sensable_phantom_models/meshes/tip.stl
- link torso: geometry visual mesh filename=package://saw_sensable_phantom_models/meshes/torso.stl
- link upper_arm: geometry visual mesh filename=package://saw_sensable_phantom_models/meshes/upper_arm.stl
- link wrist: geometry visual mesh filename=package://saw_sensable_phantom_models/meshes/wrist.stl

Commit message: models with launch and rviz files working for ROS1 and ROS2

File: models/urdf/omni.urdf (robot description, URDF)
Before this commit: robot phantom_omni, 7 links, 6 joints
Links:
- link base: geometry visual mesh filename=package://sensable_phantom_models/meshes/base.stl
- link lower_arm: geometry visual mesh filename=package://sensable_phantom_models/meshes/lower_arm.stl
- link stylus: geometry visual mesh filename=package://sensable_phantom_models/meshes/stylus.stl
- link tip: geometry visual mesh filename=package://sensable_phantom_models/meshes/tip.stl
- link torso: geometry visual mesh filename=package://sensable_phantom_models/meshes/torso.stl
- link upper_arm: geometry visual mesh filename=package://sensable_phantom_models/meshes/upper_arm.stl
- link wrist: geometry visual mesh filename=package://sensable_phantom_models/meshes/wrist.stl
Joints:
- joint pitch: origin xyz=0 0.0525 0 rpy=1.5708 0 0 -> xyz=0 0.0525 0 rpy=1.5707 0 0
- joint yaw: axis 0 -1 0 -> 0 1 0

Commit message: Improved homing, tested on FireWire Sensable Omni and Ethernet 3DS Touch.  Changed colors for model

File: models/urdf/omni.urdf (robot description, URDF)
Before this commit: robot phantom_omni, 7 links, 6 joints
Joints:
- joint yaw: axis 0 1 0 -> 0 -1 0
